File: input/EAGLE/axiom_beta_power_board_v0.37_r1.2/axiom_beta_power_board_v0.37_r1.2.brd (EAGLE design)
At the start: 101.6 x 57.1 mm, 329 parts, among them Q1 NX3008NBKT, U1 PIC16F15325-JQ, U10 AP7312-3333W6-7, U11 AP7312-3333W6-7, U12 AP7312-3333W6-7, U13 AP7312-3333W6-7, U14 PAC1720, U15 PAC1720, U16 PAC1720, U17 PAC1720, U18 PAC1720, U19 PAC1720, U2 TPS82130SIL-GM, U20 PAC1720, U21 PAC1720, U22 PAC1720, U23 PAC1720, U24 PAC1720, U25 PCA9306GM, U26 SC202A, U27 TS3A4751, U28 IP4251CZ16-8-TTL, U29 LM75BGD, U3 TPS82130SIL-GM, U30 PCA9306GM, U31 NCP715, U4 PCA9306GM, U5 PCA9306GM, U6 MCP23018-E/MJ, U7 MCP23018-E/MJ, U8 MCP23018-E/MJ, U9 MCP23018-E/MJ, X1 PICO-SPOX-5

Commit message: - Added component position data
Parts:
- R10, R2: value 102k -> RB
- R12: value 28k -> RD
- R14, R18, R33, R35, R39, R41, R43, R45, R47, R49, R6: value 180k -> RB
- R16, R20, R34, R36, R40, R42, R44, R46, R48, R50, R8: value 25k5 -> RD
- R22, R30: value 147k -> RB
- R24, R32: value 102k -> RD
- R26: value 124k -> RB
- R28: value 19k6 -> RD
- R4: value 20k -> RD
