File: input/EAGLE/axiom_beta_interface_dummy_v0.13_r1.3/axiom_beta_interface_dummy_v0.13_r1.3.brd (EAGLE design)
At the start: 57.1 x 57.1 mm, 33 parts

Commit message: updated all boards and gerbers
Other:
- board text added: "Copyright (C) 2015-2020 H.Pötzl Licensed under CERN OHL v1.2"
- board text removed: "Copyright (C) 2015 Herbert Pötzl Licensed under CERN OHL v.1.2"
Changed lines of the file:
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@@
 <setting verticaltext="up"/>
 </settings>
-<grid distance="0.25" unitdist="mm" unit="mm" style="lines" multiple="1" display="yes" altdistance="0.5" altunitdist="mm" altunit="mm"/>
+<grid distance="0.05" unitdist="inch" unit="inch" style="lines" multiple="1" display="yes" altdistance="0.025" altunitdist="inch" altunit="inch"/>
 <layers>
 <layer number="1" name="Top" color="16" fill="1" visible="yes" active="yes"/>
@@
 <wire x1="38.1" y1="-37.846" x2="38.1" y2="-38.354" width="0.1524" layer="48"/>
 <wire x1="37.846" y1="-38.1" x2="38.354" y2="-38.1" width="0.1524" layer="48"/>
-<text x="-7.67" y="-6.22" size="0.7112" layer="53" font="vector" ratio="15" align="center-left">Copyright (C) 2015 Herbert Pötzl
-Licensed under CERN OHL v.1.2</text>
+<text x="-7.67" y="-6.22" size="0.7112" layer="53" font="vector" ratio="15" align="center-left">Copyright (C) 2015-2020 H.Pötzl
+Licensed under CERN OHL v1.2</text>
 <text x="0" y="6.985" size="1.08" layer="53" font="vector" ratio="15" align="center">Dummy Interface Board</text>
 <text x="3.095" y="-3.165" size="1.905" layer="53" font="vector" ratio="14" rot="SR0">beta</text>
