File: input/EAGLE/axiom_beta_main_board_v0.37_r1.1/axiom_beta_main_board_v0.37_r1.1.brd (EAGLE design)
At the start: 111.8 x 57.1 mm, 124 parts, among them T1 NX3008NBKT, T2 NX3008NBKT, U1 PCA9540BDP, U2 PIC16F1718-I/MV, U3 PIC16F1718-I/MV

Commit message: updated all boards and gerbers
Parts:
- moved LOGO1 2.40 mm to (-15.4, -23.4)
Other:
- board text added: "Copyright (C) 2015-2020 H.Pötzl Licensed under CERN OHL v1.2"
- board text removed: "Copyright (C) 2015-2020 Herbert Pötzl Licensed under CERN OHL v.1.2"
