File: input/EAGLE/axiom_beta_sensor_cmv12000_tht_v0.16_r1.5c/axiom_beta_sensor_cmv12000_tht_v0.16_r1.5c.brd (EAGLE design)
At the start: 57.1 x 57.1 mm, 159 parts, among them U1 TLV431DCK, U2 TLV431DCK, U3 MIC47050, U4 SN74AVC4T774RSV, U5 SN74AVC4T774RSV, U6 SN74AVC4T774RSV, U7 LM75BGD

Commit message: updated all boards and gerbers
Other:
- board text added: "Copyright (C) 2015-2020 H.Pötzl Licensed under CERN OHL v1.2"
- board text removed: "Copyright (C) 2015-2017 H.Pötzl Licensed under CERN OHL v1.2"
Changed lines of the file:
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@@
 <wire x1="11.2" y1="-4.69" x2="8.66" y2="-7.23" width="0.127" layer="20" curve="-90"/>
 <text x="0" y="24.765" size="1.016" layer="53" font="vector" ratio="15" align="center">AXIOM Beta CMV12000 Sensor Board</text>
-<text x="0" y="-19.685" size="1.016" layer="53" font="vector" ratio="15" align="center">Copyright (C) 2015-2017 H.Pötzl
+<text x="0" y="-19.685" size="1.016" layer="53" font="vector" ratio="15" align="center">Copyright (C) 2015-2020 H.Pötzl
 Licensed under CERN OHL v1.2</text>
 <text x="-24.13" y="20.32" size="1.016" layer="53" font="vector" ratio="15" align="center">V0.16
