File: input/base_variant/axiom_beta_power_board_v0.37_r1.2/axiom_beta_power_board_v0.37_r1.2.brd (EAGLE design)
At the start: 101.6 x 57.1 mm, 329 parts, among them Q1 NX3008NBKT, U1 PIC16F15325-JQ, U10 AP7312-3333W6-7, U11 AP7312-3333W6-7, U12 AP7312-3333W6-7, U13 AP7312-3333W6-7, U14 PAC1720, U15 PAC1720, U16 PAC1720, U17 PAC1720, U18 PAC1720, U19 PAC1720, U2 TPS82130SIL-GM, U20 PAC1720, U21 PAC1720, U22 PAC1720, U23 PAC1720, U24 PAC1720, U25 PCA9306GM, U26 SC202A, U27 TS3A4751, U28 IP4251CZ16-8-TTL, U29 LM75BGD, U3 TPS82130SIL-GM, U30 PCA9306GM, U31 NCP715, U4 PCA9306GM, U5 PCA9306GM, U6 MCP23018-E/MJ, U7 MCP23018-E/MJ, U8 MCP23018-E/MJ, U9 MCP23018-E/MJ, X1 PICO-SPOX-5

Commit message: updated all boards and gerbers
Other:
- board text added: "Copyright (C) 2015-2020 H.Pötzl Licensed under CERN OHL v1.2"
- board text removed: "Copyright (C) 2015-2020 Herbert Pötzl Licensed under CERN OHL v.1.2"
Changed lines of the file:
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@@
 <layer number="25" name="tNames" color="7" fill="1" visible="yes" active="yes"/>
 <layer number="26" name="bNames" color="7" fill="1" visible="yes" active="yes"/>
-<layer number="27" name="tValues" color="11" fill="1" visible="no" active="yes"/>
-<layer number="28" name="bValues" color="11" fill="1" visible="no" active="yes"/>
+<layer number="27" name="tValues" color="11" fill="1" visible="yes" active="yes"/>
+<layer number="28" name="bValues" color="11" fill="1" visible="yes" active="yes"/>
 <layer number="29" name="tStop" color="7" fill="3" visible="yes" active="yes"/>
 <layer number="30" name="bStop" color="7" fill="6" visible="yes" active="yes"/>
@@
 <circle x="-46.99" y="-24.765" radius="2.54" width="0" layer="40"/>
 <wire x1="-50.8" y1="-28.575" x2="-50.8" y2="28.575" width="0.000003125" layer="20"/>
-<text x="-30.7975" y="-1.27" size="0.8128" layer="53" font="vector" ratio="15" align="center-left">Copyright (C) 2015-2020 Herbert Pötzl
-Licensed under CERN OHL v.1.2</text>
+<text x="-30.7975" y="-1.27" size="0.8636" layer="53" font="vector" ratio="15" align="center-left">Copyright (C) 2015-2020 H.Pötzl
+Licensed under CERN OHL v1.2</text>
 <text x="20.574" y="1.2065" size="1.27" layer="53" font="vector" ratio="16" align="center">AXIOM Beta
 Power Board</text>
