File: input/EAGLE/test_strip_v0.1_r1.2/test_strip_v0.1_r1.2.brd (EAGLE design)
At the start: 121.9 x 176.5 mm, 8 parts, among them X1 BU-SMA-E-ND, X2 BU-SMA-E-ND, X3 BU-SMA-E-ND, X4 BU-SMA-E-ND, X5 BU-SMA-E-ND, X6 BU-SMA-E-ND, X7 BU-SMA-E-ND, X8 BU-SMA-E-ND

Commit message: commited updated gerbers
Routing:
- net SIGA_P: track 578.2 -> 580.0 mm
- net SIGA_N: track 579.2 -> 580.1 mm
Other:
- board text added: "V0.1 R1.2"
